File: CCM_0006_Magnetic_Field_Sensor/hardware/CCM0006.brd (EAGLE design)
At the start: 49.4 x 25.4 mm, 31 parts, among them IC1 AD654, IC2 LM6061, IC4 AD8436, X1 22-23-2021

Commit message: added resources for updating the firmware of the reflow oven
Parts:
- IC2: value LM6061 -> LMC6061
- R1: value 10k -> 1k
Changed lines of the file:
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@@
 <attribute name="NAME" x="23.876" y="7.62" size="0.6096" layer="25" rot="R180"/>
 </element>
-<element name="R1" library="ic" package="0402" value="10k" x="26.543" y="3.556" smashed="yes" rot="R90">
+<element name="R1" library="ic" package="0402" value="1k" x="26.543" y="3.556" smashed="yes" rot="R90">
 <attribute name="NAME" x="26.035" y="4.953" size="0.6096" layer="25" font="vector"/>
 </element>
@@
 <attribute name="NAME" x="27.051" y="-10.033" size="0.6096" layer="26" font="vector" rot="MR90"/>
 </element>
-<element name="IC2" library="analog-devices" package="SO8" value="LM6061" x="17.78" y="-4.191" smashed="yes" rot="R270">
+<element name="IC2" library="analog-devices" package="SO8" value="LMC6061" x="17.78" y="-4.191" smashed="yes" rot="R270">
 <attribute name="OC_NEWARK" value="unknown" x="17.78" y="-4.191" size="1.778" layer="27" rot="R270" display="off"/>
 <attribute name="MPN" value="" x="17.78" y="-4.191" size="1.778" layer="27" rot="R270" display="off"/>
