File: PiezoAmp/PiezoAmpHVDCv3.sch (EAGLE design)
At the start: 35 parts, among them IC1 LM101N, Q1 IRF512, Q2 IRF512, Q3 2N3904, U1 RXX100, X1 MAB32

Commit message: Trying to clean up
Clean up, add Piezo sent to DirtyPCB
Parts:
- added POT: 10k, pinhead:PINHD-1X3
- added R13, R14: 100k, rcl:R-EU_0204/5
- added R17: 4k7, rcl:R-EU_0204/5
- D1, D2, D3, D4: value 1N4148DO35-7 -> 1N4148
- Q1, Q2: value IRF512 -> IRFU214
Connections:
- new net N$10: IC1.-IN, R13.2, R14.1
- new net N$13: POT.2, R14.2
- new net N$17: POT.3, R17.1
- net +15V: now also R17.2
- net GND: now also POT.1
- net N$1: now also R13.1; no longer IC1.-IN
Other:
- moved on the sheet: C4, JP1
Changed lines of the file:
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@@
 <?xml version="1.0" encoding="utf-8"?>
 <!DOCTYPE eagle SYSTEM "eagle.dtd">
-<eagle version="6.5.0">
+<eagle version="6.6.0">
 <drawing>
 <settings>
@@
 <parts>
 <part name="IC1" library="linear" deviceset="LM101" device="N"/>
-<part name="D1" library="diode" deviceset="1N4148" device="DO35-7"/>
-<part name="D2" library="diode" deviceset="1N4148" device="DO35-7"/>
-<part name="D3" library="diode" deviceset="1N4148" device="DO35-7"/>
-<part name="D4" library="diode" deviceset="1N4148" device="DO35-7"/>
+<part name="D1" library="diode" deviceset="1N4148" device="DO35-7" value="1N4148"/>
+<part name="D2" library="diode" deviceset="1N4148" device="DO35-7" value="1N4148"/>
+<part name="D3" library="diode" deviceset="1N4148" device="DO35-7" value="1N4148"/>
+<part name="D4" library="diode" deviceset="1N4148" device="DO35-7" value="1N4148"/>
 <part name="D5" library="diode" deviceset="ZENER-DIODE" device="DO34-7"/>
 <part name="R1" library="rcl" deviceset="R-EU_" device="0204/7" value="5.1k"/>
@@
 <part name="GND6" library="supply1" deviceset="GND" device=""/>
 <part name="X1" library="con-vg" deviceset="MAB32" device=""/>
-<part name="Q1" library="transistor-power" deviceset="IRF512" device=""/>
-<part name="Q2" library="transistor-power" deviceset="IRF512" device=""/>
+<part name="Q1" library="transistor-power" deviceset="IRF512" device="" value="IRFU214"/>
+<part name="Q2" library="transistor-power" deviceset="IRF512" device="" value="IRFU214"/>
 <part name="U1" library="custom_parts" deviceset="RXX100" device=""/>
 <part name="P+3" library="supply1" deviceset="+15V" device=""/>
@@
 <part name="C7" library="rcl" deviceset="CPOL-EU" device="SANYO_F8" value="47u/16V"/>
 <part name="R12" library="rcl" deviceset="R-EU_" device="0204/7" value="5k"/>
+<part name="R13" library="rcl" deviceset="R-EU_" device="0204/5" value="100k"/>
+<part name="POT" library="pinhead" deviceset="PINHD-1X3" device="" value="10k"/>
+<part name="GND9" library="supply1" deviceset="GND" device=""/>
+<part name="R14" library="rcl" deviceset="R-EU_" device="0204/5" value="100k"/>
+<part name="P+4" library="supply1" deviceset="+15V" device=""/>
+<part name="R17" library="rcl" deviceset="R-EU_" device="0204/5" value="4k7"/>
 </parts>
 <sheets>
@@
 <instance part="R7" gate="G$1" x="50.8" y="30.48"/>
 <instance part="R8" gate="G$1" x="66.04" y="22.86" rot="R270"/>
-<instance part="JP1" gate="G$1" x="27.94" y="71.12" rot="R180"/>
+<instance part="JP1" gate="G$1" x="22.86" y="71.12" rot="R180"/>
 <instance part="JP2" gate="G$1" x="160.02" y="27.94"/>
 <instance part="R9" gate="G$1" x="129.54" y="22.86"/>
@@
 <instance part="C2" gate="G$1" x="20.32" y="55.88"/>
 <instance part="C3" gate="G$1" x="25.4" y="35.56" rot="R180"/>
-<instance part="C4" gate="G$1" x="43.18" y="88.9"/>
+<instance part="C4" gate="G$1" x="66.04" y="91.44"/>
 <instance part="C5" gate="G$1" x="78.74" y="38.1" rot="R90"/>
 <instance part="C6" gate="G$1" x="137.16" y="20.32"/>
 <instance part="GND1" gate="1" x="50.8" y="15.24"/>
 <instance part="GND2" gate="1" x="144.78" y="12.7"/>
-<instance part="GND3" gate="1" x="43.18" y="76.2"/>
-<instance part="GND4" gate="1" x="38.1" y="60.96"/>
+<instance part="GND3" gate="1" x="66.04" y="81.28"/>
+<instance part="GND4" gate="1" x="33.02" y="63.5"/>
 <instance part="GND5" gate="1" x="20.32" y="45.72"/>
 <instance part="P+1" gate="1" x="50.8" y="55.88" rot="R90"/>
@@
 <instance part="C7" gate="G$1" x="66.04" y="0"/>
 <instance part="R12" gate="G$1" x="96.52" y="-22.86"/>
+<instance part="R13" gate="G$1" x="40.64" y="68.58"/>
+<instance part="POT" gate="A" x="25.4" y="83.82" rot="R180"/>
+<instance part="GND9" gate="1" x="20.32" y="76.2"/>
+<instance part="R14" gate="G$1" x="40.64" y="76.2" rot="R180"/>
+<instance part="P+4" gate="1" x="50.8" y="88.9"/>
+<instance part="R17" gate="G$1" x="40.64" y="86.36"/>
 </instances>
 <busses>
 </busses>
 <nets>
-<net name="N$1" class="0">
-<segment>
-<wire x1="30.48" y1="71.12" x2="50.8" y2="71.12" width="0.1524" layer="91"/>
-<pinref part="JP1" gate="G$1" pin="2"/>
-<pinref part="IC1" gate="A" pin="-IN"/>
-</segment>
-</net>
 <net name="N$7" class="0">
 <segment>
@@
 <net name="HV" class="0">
 <segment>
-<wire x1="43.18" y1="91.44" x2="43.18" y2="93.98" width="0.1524" layer="91"/>
-<wire x1="43.18" y1="93.98" x2="91.44" y2="93.98" width="0.1524" layer="91"/>
+<wire x1="66.04" y1="93.98" x2="91.44" y2="93.98" width="0.1524" layer="91"/>
 <pinref part="C4" gate="G$1" pin="1"/>
 <pinref part="R10" gate="G$1" pin="2"/>
@@
 </segment>
 <segment>
-<wire x1="43.18" y1="78.74" x2="43.18" y2="83.82" width="0.1524" layer="91"/>
-<wire x1="15.24" y1="83.82" x2="43.18" y2="83.82" width="0.1524" layer="91"/>
-<junction x="43.18" y="83.82"/>
+<wire x1="66.04" y1="83.82" x2="66.04" y2="86.36" width="0.1524" layer="91"/>
 <pinref part="GND3" gate="1" pin="GND"/>
 <pinref part="C4" gate="G$1" pin="2"/>
-<pinref part="X1" gate="G$1" pin="1"/>
-</segment>
-<segment>
-<wire x1="38.1" y1="63.5" x2="38.1" y2="68.58" width="0.1524" layer="91"/>
-<wire x1="38.1" y1="68.58" x2="30.48" y2="68.58" width="0.1524" layer="91"/>
-<pinref part="GND4" gate="1" pin="GND"/>
-<pinref part="JP1" gate="G$1" pin="1"/>
 </segment>
 <segment>
@@
 <pinref part="GND6" gate="1" pin="GND"/>
 <wire x1="91.44" y1="55.88" x2="91.44" y2="50.8" width="0.1524" layer="91"/>
+</segment>
+<segment>
+<pinref part="JP1" gate="G$1" pin="1"/>
+<pinref part="GND4" gate="1" pin="GND"/>
+<wire x1="33.02" y1="66.04" x2="33.02" y2="68.58" width="0.1524" layer="91"/>
+<wire x1="33.02" y1="68.58" x2="25.4" y2="68.58" width="0.1524" layer="91"/>
+</segment>
+<segment>
+<pinref part="X1" gate="G$1" pin="1"/>
+<pinref part="GND9" gate="1" pin="GND"/>
+<wire x1="15.24" y1="83.82" x2="20.32" y2="83.82" width="0.1524" layer="91"/>
+<wire x1="20.32" y1="83.82" x2="20.32" y2="78.74" width="0.1524" layer="91"/>
+<pinref part="POT" gate="A" pin="1"/>
+<wire x1="27.94" y1="81.28" x2="27.94" y2="78.74" width="0.1524" layer="91"/>
+<wire x1="27.94" y1="78.74" x2="20.32" y2="78.74" width="0.1524" layer="91"/>
+<junction x="20.32" y="78.74"/>
 </segment>
 </net>
@@
 <junction x="66.04" y="7.62"/>
 </segment>
+<segment>
+<pinref part="R17" gate="G$1" pin="2"/>
+<pinref part="P+4" gate="1" pin="+15V"/>
+<wire x1="45.72" y1="86.36" x2="50.8" y2="86.36" width="0.1524" layer="91"/>
+</segment>
 </net>
 <net name="-15V" class="0">
@@
 </segment>
 </net>
+<net name="N$1" class="0">
+<segment>
+<pinref part="JP1" gate="G$1" pin="2"/>
+<wire x1="25.4" y1="71.12" x2="35.56" y2="71.12" width="0.1524" layer="91"/>
+<pinref part="R13" gate="G$1" pin="1"/>
+<wire x1="35.56" y1="71.12" x2="35.56" y2="68.58" width="0.1524" layer="91"/>
+</segment>
+</net>
+<net name="N$10" class="0">
+<segment>
+<pinref part="R13" gate="G$1" pin="2"/>
+<wire x1="45.72" y1="68.58" x2="48.26" y2="68.58" width="0.1524" layer="91"/>
+<wire x1="48.26" y1="68.58" x2="48.26" y2="71.12" width="0.1524" layer="91"/>
+<pinref part="IC1" gate="A" pin="-IN"/>
+<wire x1="48.26" y1="71.12" x2="50.8" y2="71.12" width="0.1524" layer="91"/>
+<pinref part="R14" gate="G$1" pin="1"/>
+<wire x1="45.72" y1="76.2" x2="48.26" y2="76.2" width="0.1524" layer="91"/>
+<wire x1="48.26" y1="76.2" x2="48.26" y2="71.12" width="0.1524" layer="91"/>
+<junction x="48.26" y="71.12"/>
+</segment>
+</net>
+<net name="N$13" class="0">
+<segment>
+<pinref part="R14" gate="G$1" pin="2"/>
+<wire x1="35.56" y1="76.2" x2="35.56" y2="83.82" width="0.1524" layer="91"/>
+<pinref part="POT" gate="A" pin="2"/>
+<wire x1="35.56" y1="83.82" x2="27.94" y2="83.82" width="0.1524" layer="91"/>
+</segment>
+</net>
+<net name="N$17" class="0">
+<segment>
+<pinref part="POT" gate="A" pin="3"/>
+<pinref part="R17" gate="G$1" pin="1"/>
+<wire x1="27.94" y1="86.36" x2="35.56" y2="86.36" width="0.1524" layer="91"/>
+</segment>
+</net>
