File: CCM_0008_Coil_Driver/coil_driver.brd (EAGLE design)
At the start: 177.8 x 101.6 mm, 203 parts, among them IC1 AD8675, IC10 AD8675, IC11 AD825, IC12 AD825, IC13 AD825, IC14 AD825, IC15 AD825, IC16 AD825, IC17 BUF634U, IC2 AD797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

Commit message: Added CAD and docs for CCM_0008
Parts:
- C2, C4: value 0.1uF -> 0.1u
- C22, C72: value 100nF -> 0.1u
Changed lines of the file:
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@@
 <attribute name="VALUE" x="157.988" y="5.715" size="1.27" layer="27" ratio="10" rot="R90"/>
 </element>
-<element name="C2" library="acrooptics" package="0603" value="0.1uF" x="151.765" y="7.366" smashed="yes" rot="R90">
+<element name="C2" library="acrooptics" package="0603" value="0.1u" x="151.765" y="7.366" smashed="yes" rot="R90">
 <attribute name="NAME" x="151.257" y="9.144" size="0.6096" layer="25" font="vector" ratio="15"/>
 <attribute name="VALUE" x="153.543" y="5.715" size="0.6096" layer="27" font="vector" ratio="20" rot="R90"/>
@@
 <attribute name="VALUE" x="170.688" y="5.715" size="1.27" layer="27" ratio="10" rot="R90"/>
 </element>
-<element name="C4" library="acrooptics" package="0603" value="0.1uF" x="172.72" y="7.366" smashed="yes" rot="R90">
+<element name="C4" library="acrooptics" package="0603" value="0.1u" x="172.72" y="7.366" smashed="yes" rot="R90">
 <attribute name="NAME" x="171.577" y="5.588" size="0.6096" layer="25" font="vector" ratio="15" rot="R90"/>
 <attribute name="VALUE" x="174.498" y="5.715" size="0.6096" layer="27" font="vector" ratio="20" rot="R90"/>
@@
 <attribute name="VALUE" x="71.755" y="15.24" size="1.27" layer="27"/>
 </element>
-<element name="C72" library="acrooptics" package="0603" value="100nF" x="98.1075" y="20.955" smashed="yes" rot="R90">
+<element name="C72" library="acrooptics" package="0603" value="0.1u" x="98.1075" y="20.955" smashed="yes" rot="R90">
 <attribute name="NAME" x="97.3455" y="22.733" size="0.6096" layer="25" font="vector" ratio="15"/>
 <attribute name="VALUE" x="99.8855" y="19.304" size="0.6096" layer="27" font="vector" ratio="20" rot="R90"/>
@@
 <attribute name="VALUE" x="102.87" y="15.24" size="1.27" layer="27"/>
 </element>
-<element name="C22" library="acrooptics" package="0603" value="100nF" x="129.2225" y="20.955" smashed="yes" rot="R90">
+<element name="C22" library="acrooptics" package="0603" value="0.1u" x="129.2225" y="20.955" smashed="yes" rot="R90">
 <attribute name="NAME" x="128.397" y="22.6695" size="0.6096" layer="25" font="vector" ratio="15"/>
 <attribute name="VALUE" x="131.0005" y="19.304" size="0.6096" layer="27" font="vector" ratio="20" rot="R90"/>

Commit message: CCM_0008: fixed current monitor schematic wiring error, prototype run current-monitor output will rail if not fixed in hardware.
Connections:
- removed net N$24: IC6.6, R27.2
- new net N$6: IC6.2, IC6.6, R27.2
- net GND: no longer IC6.2
Routing:
- net N$6: track 0.00 -> 8.59 mm
- net N$24: track 2.86 -> 0.00 mm
- net GND: track 160.1 -> 158.0 mm, vias 49 -> 48
Changed lines of the file:
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@@
 <contactref element="C92" pad="1"/>
 <contactref element="C93" pad="1"/>
-<contactref element="IC6" pad="2"/>
 <contactref element="S3" pad="3"/>
 <wire x1="24.003" y1="59.563" x2="24.003" y2="61.595" width="0.4064" layer="1"/>
@@
 <wire x1="6.985" y1="30.226" x2="5.715" y2="30.226" width="0.4064" layer="1"/>
 <via x="5.715" y="30.226" extent="1-16" drill="0.5"/>
-<wire x1="10.16" y1="25.587" x2="10.16" y2="23.495" width="0.4064" layer="1"/>
-<via x="10.16" y="23.495" extent="1-16" drill="0.5"/>
 <wire x1="2.286" y1="71.12" x2="2.286" y2="69.215" width="0.4064" layer="1"/>
 <wire x1="15.875" y1="46.736" x2="15.875" y2="45.085" width="0.4064" layer="1"/>
@@
 <via x="8.89" y="36.83" extent="1-16" drill="0.5"/>
 </signal>
-<signal name="N$24">
-<contactref element="R27" pad="2"/>
-<contactref element="IC6" pad="6"/>
-<wire x1="8.89" y1="20.387" x2="8.89" y2="17.526" width="0.4064" layer="1"/>
-</signal>
 <signal name="N$25">
 <contactref element="R27" pad="1"/>
@@
 <wire x1="8.89" y1="28.448" x2="8.89" y2="25.587" width="0.4064" layer="1"/>
 </signal>
+<signal name="N$6">
+<contactref element="IC6" pad="2"/>
+<contactref element="R27" pad="2"/>
+<contactref element="IC6" pad="6"/>
+<wire x1="8.89" y1="20.387" x2="8.89" y2="17.526" width="0.4064" layer="1"/>
+<wire x1="10.16" y1="25.587" x2="10.16" y2="23.749" width="0.4064" layer="1"/>
+<wire x1="10.16" y1="23.749" x2="8.89" y2="22.479" width="0.4064" layer="1"/>
+<wire x1="8.89" y1="22.479" x2="8.89" y2="20.387" width="0.4064" layer="1"/>
+</signal>
 </signals>
