File: CCM_0007_F50_Cryocooler_Controller/v2/hardware/F50_cryocooler_controller.brd (EAGLE design)
At the start: 140 x 100 mm, 50 parts, among them IC1 74LVC1G79DBV, IC2 MCP601OT, Q2 IRLL024, Q3 IRLL024, U1 MAX4466EXK+T, U3 PHOTON_WITH_HEADERS, X2 BNCPTH

Commit message: CCM_0007: finished layout of v2.
Parts:
- removed IC1: 74LVC1G79DBV, 74xx-little-de:SOT23-5
- removed IC2: MCP601OT, linear:SOT23-5
- removed R14, R15, R25: 10k, acrooptics:0603
- removed U$1, U$2, U$3: BNCPTH, SparkFun:BNC
- added D1, D7: (no value), acrooptics:LED0603
- added R3, R6, R7, R8, R9: 1k, acrooptics:0603
- added U2: MCP601OT, linear:SOT23-5
- added U4: 74LVC1G79DBV, 74xx-little-de:SOT23-5
- added X3: 22-23-2021, con-molex:22-23-2021
- added X4, X5: BNCPTH, SparkFun:BNC
- R13: value 10k -> 1k
- X1: value (none) -> Male DB15
- moved R20 202.0 mm to (25.4, 38.0), turned to 270 degrees
- moved C11 201.3 mm to (37.2, 43.2), turned to 270 degrees
- moved R18 196.2 mm to (37.2, 46.8), turned to 90 degrees
- moved R19 191.8 mm to (23.0, 32.5)
- moved D6 174.1 mm to (23.0, 35.0), turned to 270 degrees
- moved D2 158.1 mm to (40.0, 43.2), turned to 270 degrees
- moved D3 143.7 mm to (18.0, 27.0), turned to 270 degrees
- moved R17 141.1 mm to (67.0, 40.4)
- moved R16 135.9 mm to (67.0, 38.7), turned to 180 degrees
- moved Q3 126.7 mm to (23.0, 27.0), turned to 180 degrees
- moved R13 89.0 mm to (15.2, 25.2), turned to 90 degrees
- moved R23 66.5 mm to (36.5, 51.2), turned to 180 degrees
- moved R24 66.2 mm to (36.5, 49.5), turned to 180 degrees
- moved R12 60.1 mm to (130.0, 23.0), turned to 90 degrees
- moved R11 49.3 mm to (67.0, 20.9)
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Connections:
- new net N$12: R6.2, X1.3
- new net N$16: R3.2, X1.5
- new net N$17: D1.C, R13.2
- new net N$18: D7.C, R9.2
- new net N$6: R8.1, X1.10
- new net N$9: R7.2, X1.1
- net 3.3V: now also U2.5; no longer IC2.5, R13.2, R14.2, R15.2, R25.2
- net APPLIED: now also D7.A, X3.1; no longer X2.GND
- net CLOCK: now also U4.2; no longer IC1.2
- net CMD: now also U4.4, X3.2; no longer IC1.4, X2.S
- net GND: now also R13.1, R9.1, U2.2, U2.3, U4.3, X2.GND, X4.GND, X5.GND; no longer IC1.3, IC2.2, IC2.3, U$1.GND, U$2.GND, U$3.GND
- net HELIUM_AFTER_COOLER_TEMP_ALARM: now also R3.1; no longer R15.1, X1.5
- net HELIUM_DISCHARGE_TEMP_ALARM: now also R6.1; no longer R14.1, X1.3
- net N$1: now also X4.S; no longer U$3.S
- net N$14: now also U4.5; no longer IC1.5
- net N$15: now also U2.1; no longer IC2.1
- net N$8: now also U2.4; no longer IC2.4
- net PRESSURE_ALARM: now also R7.1; no longer R13.1, X1.1
- net RESET: now also D1.A
- net STATE_TO_LATCH: now also U4.1; no longer IC1.1
- net SYNC_OUT: now also X2.S; no longer U$1.S
- net TRIGGER_OUT: now also X5.S; no longer U$2.S
- net WATER_TEMP_ALARM: now also R8.2; no longer R25.1, X1.10
Routing:
- net RESET: track 0.00 -> 123.8 mm
- net APPLIED: track 0.00 -> 99.5 mm
- net CMD: track 0.00 -> 91.7 mm, vias 0 -> 1
- net N$9: track 0.00 -> 72.7 mm, vias 0 -> 1
- net N$12: track 0.00 -> 67.5 mm
- net N$6: track 0.00 -> 66.6 mm
- net +24V: track 0.00 -> 66.1 mm, vias 0 -> 3
- net CLOCK: track 0.00 -> 65.6 mm, vias 0 -> 1
- net N$16: track 0.00 -> 61.8 mm
- net N$7: track 0.00 -> 57.4 mm
- net STATE_TO_LATCH: track 0.00 -> 56.8 mm, vias 0 -> 1
- net N$15: track 0.00 -> 54.3 mm, vias 0 -> 1
- net GND: track 13.5 -> 44.0 mm, vias 6 -> 16
- net N$19: track 0.00 -> 14.6 mm
- net SYNC_OUT: track 0.00 -> 13.9 mm
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Other:
- board size 140 x 100 mm -> 141.5 x 49 mm
- board text added: "microphone"
- board text added: "trigger out"
- board text added: "volume out"
