File: CCM_0009_Precision_Coil_Driver/CCM_0009.sch (EAGLE design)
At the start: 130 parts, among them Q1 TIP29, Q2 TIP30, Q5 TIP29, Q6 TIP30, Q7 TIP29, Q8 TIP30, U1 ADA4898-2, U10 ADA4898-2, U11 AD8276, U12 AD4898-1, U13 BUF634, U14 ADA4898-2, U15 AD8276, U16 AD4898-1, U2 AD8276, U3 BUF634, U4 AD4898-1, U9 BUF634, X1 1-227161-0, X10 22-23-2021, X11 22-23-2031, X12 22-23-2031, X13 1-227161-0, X14 22-23-2021, X15 22-23-2031, X16 22-23-2031, X2 22-23-2021, X4 22-23-2031, X5 22-23-2031, X6 22-23-2031, X7 22-23-2031, X9 1-227161-0

Commit message: production files for CCM_0009
Parts:
- R27, R40, R6: value (none) -> DNI
Changed lines of the file:
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@@
 <part name="SUPPLY5" library="supply2" deviceset="GND" device=""/>
 <part name="RO" library="noah" deviceset="LT030" device="" value="1.00"/>
-<part name="R6" library="noah" deviceset="RESISTOR" device="2512"/>
+<part name="R6" library="noah" deviceset="RESISTOR" device="2512" value="DNI"/>
 <part name="X13" library="con-coax" deviceset="?227161*" device="1-" technology="-0"/>
 <part name="TP8" library="Fitch" deviceset="TESTPOINT" device=""/>
@@
 <part name="SUPPLY24" library="supply2" deviceset="GND" device=""/>
 <part name="RO3" library="noah" deviceset="LT030" device="" value="1.00"/>
-<part name="R40" library="noah" deviceset="RESISTOR" device="2512"/>
+<part name="R40" library="noah" deviceset="RESISTOR" device="2512" value="DNI"/>
 <part name="X9" library="con-coax" deviceset="?227161*" device="1-" technology="-0"/>
 <part name="TP6" library="Fitch" deviceset="TESTPOINT" device=""/>
@@
 <part name="SUPPLY18" library="supply2" deviceset="GND" device=""/>
 <part name="RO2" library="noah" deviceset="LT030" device="" value="1.00"/>
-<part name="R27" library="noah" deviceset="RESISTOR" device="2512"/>
+<part name="R27" library="noah" deviceset="RESISTOR" device="2512" value="DNI"/>
 <part name="FRAME2" library="frames" library_urn="urn:adsk.eagle:library:229" deviceset="A4L-LOC" device=""/>
 <part name="X5" library="con-molex" deviceset="22-23-2031" device=""/>
@@
 <instance part="R6" gate="G$1" x="200.66" y="100.965" smashed="yes">
 <attribute name="NAME" x="199.39" y="97.3836" size="1.778" layer="95"/>
-<attribute name="VALUE" x="196.85" y="97.663" size="1.778" layer="96"/>
+<attribute name="VALUE" x="198.755" y="95.123" size="1.778" layer="96"/>
 </instance>
 </instances>
@@
 <instance part="R40" gate="G$1" x="200.66" y="100.965" smashed="yes">
 <attribute name="NAME" x="199.39" y="97.3836" size="1.778" layer="95"/>
-<attribute name="VALUE" x="196.85" y="97.663" size="1.778" layer="96"/>
+<attribute name="VALUE" x="199.39" y="95.123" size="1.778" layer="96"/>
 </instance>
 </instances>
@@
 <instance part="R27" gate="G$1" x="200.66" y="100.965" smashed="yes">
 <attribute name="NAME" x="199.39" y="97.3836" size="1.778" layer="95"/>
-<attribute name="VALUE" x="196.85" y="97.663" size="1.778" layer="96"/>
+<attribute name="VALUE" x="199.39" y="94.488" size="1.778" layer="96"/>
 </instance>
 </instances>
@@
 </sheet>
 </sheets>
-<errors>
-</errors>
 </schematic>
 </drawing>
