File: CCM_0009_Precision_Coil_Driver/CCM_0009.brd (EAGLE design)
At the start: 82.5 x 76.2 mm, 130 parts, among them Q1 TIP29, Q2 TIP30, Q5 TIP29, Q6 TIP30, Q7 TIP29, Q8 TIP30, U1 ADA4898-2, U10 ADA4898-2, U11 AD8276, U12 AD4898-1, U13 BUF634, U14 ADA4898-2, U15 AD8276, U16 AD4898-1, U2 AD8276, U3 BUF634, U4 AD4898-1, U9 BUF634, X1 1-227161-0, X10 22-23-2021, X11 22-23-2031, X12 22-23-2031, X13 1-227161-0, X14 22-23-2021, X15 22-23-2031, X16 22-23-2031, X2 22-23-2021, X4 22-23-2031, X5 22-23-2031, X6 22-23-2031, X7 22-23-2031, X9 1-227161-0

Commit message: production files for CCM_0009
Parts:
- R27, R40, R6: value (none) -> DNI
Changed lines of the file:
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@@
 <grid distance="0.0025" unitdist="inch" unit="inch" style="lines" multiple="10" display="yes" altdistance="0.05" altunitdist="inch" altunit="inch"/>
 <layers>
-<layer number="1" name="Top" color="4" fill="1" visible="no" active="yes"/>
+<layer number="1" name="Top" color="4" fill="1" visible="yes" active="yes"/>
 <layer number="2" name="Route2" color="1" fill="3" visible="no" active="no"/>
 <layer number="3" name="Route3" color="4" fill="3" visible="no" active="no"/>
@@
 <layer number="14" name="Route14" color="1" fill="6" visible="no" active="no"/>
 <layer number="15" name="Route15" color="4" fill="6" visible="no" active="no"/>
-<layer number="16" name="Bottom" color="1" fill="1" visible="no" active="yes"/>
-<layer number="17" name="Pads" color="2" fill="1" visible="no" active="yes"/>
-<layer number="18" name="Vias" color="2" fill="1" visible="no" active="yes"/>
-<layer number="19" name="Unrouted" color="6" fill="1" visible="no" active="yes"/>
-<layer number="20" name="Dimension" color="15" fill="1" visible="no" active="yes"/>
+<layer number="16" name="Bottom" color="1" fill="1" visible="yes" active="yes"/>
+<layer number="17" name="Pads" color="2" fill="1" visible="yes" active="yes"/>
+<layer number="18" name="Vias" color="2" fill="1" visible="yes" active="yes"/>
+<layer number="19" name="Unrouted" color="6" fill="1" visible="yes" active="yes"/>
+<layer number="20" name="Dimension" color="15" fill="1" visible="yes" active="yes"/>
 <layer number="21" name="tPlace" color="7" fill="1" visible="yes" active="yes"/>
-<layer number="22" name="bPlace" color="14" fill="1" visible="no" active="yes"/>
-<layer number="23" name="tOrigins" color="15" fill="1" visible="no" active="yes"/>
-<layer number="24" name="bOrigins" color="15" fill="1" visible="no" active="yes"/>
-<layer number="25" name="tNames" color="7" fill="1" visible="no" active="yes"/>
-<layer number="26" name="bNames" color="7" fill="1" visible="no" active="yes"/>
+<layer number="22" name="bPlace" color="14" fill="1" visible="yes" active="yes"/>
+<layer number="23" name="tOrigins" color="15" fill="1" visible="yes" active="yes"/>
+<layer number="24" name="bOrigins" color="15" fill="1" visible="yes" active="yes"/>
+<layer number="25" name="tNames" color="7" fill="1" visible="yes" active="yes"/>
+<layer number="26" name="bNames" color="7" fill="1" visible="yes" active="yes"/>
 <layer number="27" name="tValues" color="7" fill="1" visible="no" active="yes"/>
 <layer number="28" name="bValues" color="7" fill="1" visible="no" active="yes"/>
@@
 <layer number="37" name="tTest" color="7" fill="1" visible="no" active="yes"/>
 <layer number="38" name="bTest" color="7" fill="1" visible="no" active="yes"/>
-<layer number="39" name="tKeepout" color="12" fill="11" visible="no" active="yes"/>
-<layer number="40" name="bKeepout" color="1" fill="11" visible="no" active="yes"/>
-<layer number="41" name="tRestrict" color="4" fill="10" visible="no" active="yes"/>
-<layer number="42" name="bRestrict" color="1" fill="10" visible="no" active="yes"/>
+<layer number="39" name="tKeepout" color="12" fill="11" visible="yes" active="yes"/>
+<layer number="40" name="bKeepout" color="1" fill="11" visible="yes" active="yes"/>
+<layer number="41" name="tRestrict" color="4" fill="10" visible="yes" active="yes"/>
+<layer number="42" name="bRestrict" color="1" fill="10" visible="yes" active="yes"/>
 <layer number="43" name="vRestrict" color="2" fill="10" visible="no" active="yes"/>
-<layer number="44" name="Drills" color="7" fill="1" visible="no" active="yes"/>
-<layer number="45" name="Holes" color="7" fill="1" visible="no" active="yes"/>
+<layer number="44" name="Drills" color="7" fill="1" visible="yes" active="yes"/>
+<layer number="45" name="Holes" color="7" fill="1" visible="yes" active="yes"/>
 <layer number="46" name="Milling" color="3" fill="1" visible="no" active="yes"/>
 <layer number="47" name="Measures" color="7" fill="1" visible="no" active="yes"/>
@@
 <layer number="49" name="Reference" color="7" fill="1" visible="no" active="yes"/>
 <layer number="50" name="dxf" color="7" fill="1" visible="no" active="no"/>
-<layer number="51" name="tDocu" color="7" fill="1" visible="no" active="yes"/>
-<layer number="52" name="bDocu" color="7" fill="1" visible="no" active="yes"/>
+<layer number="51" name="tDocu" color="7" fill="1" visible="yes" active="yes"/>
+<layer number="52" name="bDocu" color="7" fill="1" visible="yes" active="yes"/>
 <layer number="53" name="tGND_GNDA" color="7" fill="9" visible="no" active="no"/>
 <layer number="54" name="bGND_GNDA" color="1" fill="9" visible="no" active="no"/>
@@
 <attribute name="VALUE" x="10.4775" y="53.0225" size="1.778" layer="27" rot="R90"/>
 </element>
-<element name="R6" library="noah" package="2512" value="" x="16.8275" y="58.1025" smashed="yes" rot="R90">
+<element name="R6" library="noah" package="2512" value="DNI" x="16.8275" y="58.1025" smashed="yes" rot="R90">
 <attribute name="NAME" x="16.1925" y="57.658" size="0.8128" layer="25" font="vector" ratio="12"/>
 <attribute name="VALUE" x="20.0025" y="55.5625" size="1.27" layer="27" rot="R90"/>
@@
 <attribute name="VALUE" x="35.8775" y="53.0225" size="1.778" layer="27" rot="R90"/>
 </element>
-<element name="R40" library="noah" package="2512" value="" x="42.2275" y="58.1025" smashed="yes" rot="R90">
+<element name="R40" library="noah" package="2512" value="DNI" x="42.2275" y="58.1025" smashed="yes" rot="R90">
 <attribute name="NAME" x="41.5925" y="57.658" size="0.8128" layer="25" font="vector" ratio="12"/>
 <attribute name="VALUE" x="45.4025" y="55.5625" size="1.27" layer="27" rot="R90"/>
@@
 <attribute name="VALUE" x="61.2775" y="52.3875" size="1.778" layer="27" rot="R90"/>
 </element>
-<element name="R27" library="noah" package="2512" value="" x="67.6275" y="57.4675" smashed="yes" rot="R90">
+<element name="R27" library="noah" package="2512" value="DNI" x="67.6275" y="57.4675" smashed="yes" rot="R90">
 <attribute name="NAME" x="66.9925" y="57.023" size="0.8128" layer="25" font="vector" ratio="12"/>
 <attribute name="VALUE" x="70.8025" y="54.9275" size="1.27" layer="27" rot="R90"/>

Commit message: started design of hardware TCL
Parts:
- R1: value 10.00k -> 9.000k
- renumbered R6 to RS2, RO to RS1
Changed lines of the file:
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@@
 <?xml version="1.0" encoding="utf-8"?>
 <!DOCTYPE eagle SYSTEM "eagle.dtd">
-<eagle version="8.3.0">
+<eagle version="8.3.1">
 <drawing>
 <settings>
@@
 <attribute name="VALUE" x="16.8275" y="46.355" size="1.27" layer="27" ratio="10"/>
 </element>
-<element name="R1" library="acrooptics" package="0603" value="10.00k" x="6.35" y="44.45" smashed="yes" rot="R270">
+<element name="R1" library="acrooptics" package="0603" value="9.000k" x="6.35" y="44.45" smashed="yes" rot="R270">
 <attribute name="NAME" x="6.7945" y="41.4655" size="0.8128" layer="25" font="vector" ratio="12" rot="R90"/>
 <attribute name="VALUE" x="4.572" y="46.101" size="0.6096" layer="27" font="vector" ratio="20" rot="R270"/>
@@
 <attribute name="VALUE" x="2.9845" y="46.101" size="0.6096" layer="27" font="vector" ratio="20" rot="R270"/>
 </element>
-<element name="RO" library="noah" package="LTO30" value="1.00" x="13.0175" y="55.5625" smashed="yes" rot="R90">
+<element name="RS1" library="noah" package="LTO30" value="1.00" x="13.0175" y="55.5625" smashed="yes" rot="R90">
 <attribute name="NAME" x="12.319" y="57.785" size="0.8128" layer="25" font="vector" ratio="12"/>
 <attribute name="VALUE" x="10.4775" y="53.0225" size="1.778" layer="27" rot="R90"/>
 </element>
-<element name="R6" library="noah" package="2512" value="DNI" x="16.8275" y="58.1025" smashed="yes" rot="R90">
+<element name="RS2" library="noah" package="2512" value="DNI" x="16.8275" y="58.1025" smashed="yes" rot="R90">
 <attribute name="NAME" x="16.1925" y="57.658" size="0.8128" layer="25" font="vector" ratio="12"/>
 <attribute name="VALUE" x="20.0025" y="55.5625" size="1.27" layer="27" rot="R90"/>
@@
 <contactref element="X2" pad="1"/>
 <contactref element="U4" pad="3"/>
-<contactref element="RO" pad="P$2"/>
-<contactref element="R6" pad="2"/>
+<contactref element="RS1" pad="P$2"/>
+<contactref element="RS2" pad="2"/>
 <wire x1="13.96479375" y1="60.9025" x2="16.8275" y2="60.9025" width="1.27" layer="1"/>
 <wire x1="13.96479375" y1="60.9025" x2="13.2775" y2="60.9025" width="1.27" layer="1"/>
@@
 <contactref element="U2" pad="5"/>
 <contactref element="J1" pad="2"/>
-<contactref element="RO" pad="P$1"/>
-<contactref element="R6" pad="1"/>
+<contactref element="RS1" pad="P$1"/>
+<contactref element="RS2" pad="1"/>
 <wire x1="15.054325" y1="55.3025" x2="16.8275" y2="55.3025" width="1.27" layer="1"/>
 <wire x1="15.054325" y1="55.3025" x2="13.2775" y2="55.3025" width="1.27" layer="1"/>
