File: CCM_0011_Hardware_TCL/module/module.sch (EAGLE design)
At the start: 130 parts, among them Q1 TIP29, Q2 TIP30, Q5 TIP29, Q6 TIP30, Q7 TIP29, Q8 TIP30, U1 ADA4898-2, U10 ADA4898-2, U11 AD8276, U12 AD4898-1, U13 BUF634, U14 ADA4898-2, U15 AD8276, U16 AD4898-1, U2 AD8276, U3 BUF634, U4 AD4898-1, U9 BUF634, X1 1-227161-0, X10 22-23-2021, X11 22-23-2031, X12 22-23-2031, X13 1-227161-0, X14 22-23-2021, X15 22-23-2031, X16 22-23-2031, X2 22-23-2021, X4 22-23-2031, X5 22-23-2031, X6 22-23-2031, X7 22-23-2031, X9 1-227161-0

Commit message: started design of hardware TCL
Parts:
- removed C24, C25, C26, C27, C28, C29, C30, C39, C40, C41, C42, C43, C44, C45, C46, C63, C64, C8: 0.1u, acrooptics:C0603
- removed C31, C32, C47, C48, C7, C9: 4.7u, acrooptics:C0603
- removed C33, C57: 10nF, acrooptics:C0603
- removed C34, C35, C58, C59: 1nF, acrooptics:C0603
- removed C36, C37, C60, C61: 47pF, acrooptics:C0603
- removed C38, C62: DNI, acrooptics:C0603
- removed D5, D6, D7, D8: BAV19W, AquariumLibrary:DIODE-SOD123
- removed J3, J4: (no value), acrooptics:SJ
- removed Q5, Q7: TIP29, transistor-power:TIP41C
- removed Q6, Q8: TIP30, transistor-power:TIP42C
- removed R18, R20, R22, R23, R26, R29, R31, R33, R34, R39: 1.000k, acrooptics:R0603
- removed R19, R30: 1M, acrooptics:R0603
- removed R21, R24, R32, R35: DNI, acrooptics:R0603
- removed R25, R38: 10.00k, acrooptics:R0603
- removed R27, R40: DNI, noah:RESISTOR2512
- removed RO2, RO3: 1.00, noah:LT030
- removed TP6, TP8: TESTPOINT, Fitch:TESTPOINT
- removed U10, U14: ADA4898-2, noah:ADA4898-2R
- removed U11, U15: AD8276, noah:AD8276
- removed U12, U16: AD4898-1, noah:ADA4898-1R
- removed U13, U9: BUF634, noah:BUF634
- removed X10, X14: 22-23-2021, con-molex:22-23-2021
- removed X11, X12, X15, X16, X5, X7: 22-23-2031, con-molex:22-23-2031
- removed X13, X9: 1-227161-0, con-coax:1-227161-0
Connections:
- removed net N$28: C33.1, C34.2, R18.2, R19.1, U10A.IN+
- removed net N$29: C33.2, C35.1, R19.2, R20.2, U10B.IN-
- removed net N$30: R18.1, X9.2
- removed net N$32: R20.1, X9.1
- removed net N$34: C36.1, R21.2, R22.2, U10A.IN-
- removed net N$36: C37.1, R21.1, R23.2, U10B.IN+
- removed net N$37: C37.2, R23.1, U10B.OUT, U11.+IN
- removed net N$38: C36.2, C38.1, R22.1, U10A.OUT, U11.-IN
- removed net N$39: J3.1, Q5.B, Q6.B, U9.OUT, X11-1.S, X12-1.S
- removed net N$40: D5.A, D6.C, R27.2, RO2.2, U12.IN+, X10-1.S
- removed net N$41: R24.1, U9.BW
- removed net N$42: C38.2, U11.OUT, U9.IN
- removed net N$43: R25.2, TP6.P$1, U11.REF, U12.OUT
- removed net N$44: J3.2, Q5.E, Q6.E, R27.1, RO2.1, U11.SENSE, X11-3.S, X12-3.S
- removed net N$45: R25.1, R26.1, U12.IN-
- removed net N$46: C57.1, C58.2, R29.2, R30.1, U14A.IN+
- removed net N$47: C57.2, C59.1, R30.2, R31.2, U14B.IN-
- removed net N$48: R29.1, X13.2
- removed net N$49: R31.1, X13.1
- removed net N$50: C60.1, R32.2, R33.2, U14A.IN-
- removed net N$51: C61.1, R32.1, R34.2, U14B.IN+
- removed net N$52: C61.2, R34.1, U14B.OUT, U15.+IN
- removed net N$53: C60.2, C62.1, R33.1, U14A.OUT, U15.-IN
- removed net N$54: J4.1, Q7.B, Q8.B, U13.OUT, X15-1.S, X16-1.S
- removed net N$55: D7.A, D8.C, R40.2, RO3.2, U16.IN+, X14-1.S
- removed net N$56: R35.1, U13.BW
- removed net N$57: C62.2, U13.IN, U15.OUT
- removed net N$58: R38.2, TP8.P$1, U15.REF, U16.OUT
- removed net N$59: J4.2, Q7.E, Q8.E, R40.1, RO3.1, U15.SENSE, X15-3.S, X16-3.S
- removed net N$60: R38.1, R39.1, U16.IN-
- net GND: no longer C24.1, C25.2, C26.2, C27.1, C28.1, C29.2, C30.1, C31.2, C32.1, C34.1, C35.2, C39.2, C40.1, C41.2, C42.2, C43.1, C44.1, C45.2, C46.1, C47.2, C48.1, C58.1, C59.2, C63.2, C64.1, C7.2, C8.2, C9.1, R26.2, R39.2, X10-2.S, X14-2.S, X5-2.S, X7-2.S
- net V+: no longer C25.1, C26.1, C29.1, C31.1, C39.1, C41.1, C42.1, C45.1, C47.1, C63.1, C7.1, C8.1, D5.C, D7.C, Q5.C, Q7.C, U10P.V+, U11.V+, U12.+VS, U13.V+, U14P.V+, U15.V+, U16.+VS, U9.V+, X12-2.S, X16-2.S, X5-1.S, X7-1.S
- net V-: no longer C24.2, C27.2, C28.2, C30.2, C32.2, C40.2, C43.2, C44.2, C46.2, C48.2, C64.2, C9.2, D6.A, D8.A, Q6.C, Q8.C, R24.2, R35.2, U10P.V-, U11.V-, U12.-VS, U13.V-, U14P.V-, U15.V-, U16.-VS, U9.V-, X11-2.S, X15-2.S, X5-3.S, X7-3.S
Other:
- note removed: "Power off +/-5V to +/-15V use lowest practical supply voltage to reduce output stage power dissipation"
