File: CCM_0010_Floating_H_Bridge/revB/CCM_0010.sch (EAGLE design)
At the start: 36 parts, among them IC1 ADUM5230, IC2 L78L12, IC3 HIP4080A, X1 22-23-2021, X2 22-23-2021, X3 22-23-2041, X4 22-23-2041

Commit message: Finalized design of revB of CCM_0010.  Floating H-bridge now uses a lower power driver, makes it possible to monitor the coil current, and implements an optically isolated bypass option.  This latter feature allows either the top or bottom MOT coils to be bypasses, greatly improving flexibility, while simultaneously eliminated ground loop problems with the bypass control signal.
Parts:
- added C16, C20, C31: 4.7u, acrooptics:C0603
- added C17, C18, C19, C21, C22, C26, C27, C29, C30: 0.1u, acrooptics:C0603
- added C23: 47p, acrooptics:C0603
- added C24, C28: 22p, acrooptics:C0603
- added C25: DNI, acrooptics:C0603
- added CS1: CASR15X, noah:CASR15X
- added D3: BAS70, WCSMain:DIODESOT23
- added IC10: BUF634, noah:BUF634
- added IC4: HIP4082, noah:HIP4082
- added IC5: HCNR200-300E, avago:HCNR200-300E
- added IC6: OP97, analog-devices:AD825R
- added IC7, IC9: AD820R, analog-devices:AD820R
- added IC8: AD8227, analog-devices:AD620R
- added R10: 6.8k, acrooptics:R0603
- added R11: 2.2k, acrooptics:R0603
- added R12: 33k, acrooptics:R0603
- added R13: 270, acrooptics:R0603
- added R14, R15, R19, R20: 1k, acrooptics:R0603
- added R16: 90k, acrooptics:R0603
- added R17: 842, acrooptics:R0603
- added R18: 20k, bourns:3386-W
- added R21: 100, acrooptics:R0603
- added R9: 100k, acrooptics:R0603
- added T1: 2N7002, zetex:NMOSSOT23
- added T2: MMBT3906, transistor:MMBT3906LT1-PNP-SOT23-BEC
- added TP1, TP2: TESTPOINT, noah:TESTPOINT
- added X10, X5, X6, X7, X8, X9: 22-23-2021, con-molex:22-23-2021
- C10, C13, C4: value 4.7u -> 0.1u
- C14, C5, C7, C9: value 0.1u -> 4.7u
- D1, D2: value BAV99 -> BAS70
- IC1: value ADUM5230 -> AD8226; device noah:ADUM5230 -> analog-devices:AD620R
- IC2: value L78L12 -> ADUM5230; device linear:78L12F -> noah:ADUM5230
- IC3: value HIP4080A -> UAL78L12; device noah:HIP4080A -> linear:78L12F
- R2: value 100 -> 10k
- R3: value 100 -> 20k
- R4: value 10k -> 100
- R5: value 10k -> 1k
- R6: value 100k -> 100
- R7: value 100k -> 10k
- X1: value 22-23-2021 -> 22-23-2041; device con-molex:22-23-2021 -> con-molex:22-23-2041
- X3, X4: value 22-23-2041 -> 22-23-2021; device con-molex:22-23-2041 -> con-molex:22-23-2021
Connections:
- removed net A_HIGH_GATE: IC3.AHO, X4-4.S
- removed net A_HIGH_SOURCE: C14.1, IC3.AHS, X4-3.S
- removed net A_LOW_GATE: IC3.ALO, X4-2.S
- removed net A_LOW_SOURCE: IC3.ALS, X4-1.S
- removed net B_HIGH_GATE: IC3.BHO, X3-1.S
- removed net B_HIGH_SOURCE: C15.1, IC3.BHS, X3-2.S
- removed net B_LOW_GATE: IC3.BLO, X3-3.S
- removed net B_LOW_SOURCE: IC3.BLS, X3-4.S
- new net +15V: C21.2, C3.1, C4.1, IC1.+V, IC6.+VS, R11.2, R13.2, X1-1.S
- new net -15V: C22.1, C5.2, C6.2, IC1.-V, IC6.-VS, R12.1, X1-4.S
- new net N$11: R16.2, R18.1
- new net N$12: C23.1, IC6.OUT, R10.1
- new net N$14: R10.2, R11.1, T2.B
- new net N$15: R13.1, T2.E
- new net N$18: C24.2, IC5.C2, IC7.IN-, R16.1
- new net N$19: IC5.A2, IC7.IN+
- new net N$21: IC4.BLI, R7.2, T1.D
- new net N$22: IC4.ALI, R6.2, T1.G
- new net N$25: IC10.IN, IC9.OUT
- new net N$26: C28.1, IC10.OUT, R21.1
- new net N$27: R21.2, X10-1.S
- new net N$3: D3.C, IC5.A, R12.2, T2.C
- new net N$31: C28.2, IC9.IN-, R20.2
- new net N$32: IC4.ALO, X6-1.S
- new net N$33: IC4.AHO, X7-1.S
- new net N$34: IC1.OUT, R5.1
- new net N$35: IC1.RG@1, R3.2
- new net N$36: IC1.RG@2, R3.1
- new net N$37: CS1.OUT, IC1.+, R1.2
- new net N$38: CS1.REF, IC1.-
- new net N$39: R5.2, X3-1.S
- new net N$4: C24.1, IC7.OUT, R18.2, R18.3, R19.1
- new net N$40: IC8.OUT, R20.1
- new net N$41: IC8.RG@1, R17.2
- new net N$42: IC8.RG@2, R17.1
- new net N$43: C25.1, IC9.IN+, R19.2
- new net N$44: R14.1, X9-1.S
- new net N$45: R15.1, X9-2.S
- new net N$46: IC8.-, R15.2
- new net N$47: IC8.+, R14.2
- new net N$7: R9.1, X8-1.S
- new net N$9: C23.2, IC5.C1, IC6.IN-, R9.2
- net +12V: now also C15.1, C16.1, C19.1, C20.1, C26.1, C27.1, C29.1, C30.1, C31.1, IC10.V+, IC2.VDDB, IC3.VO, IC4.AHI, IC4.BHI, IC4.VDD, IC7.+VS, IC8.+V, IC9.+VS, R7.1; no longer C10.1, C12.1, C13.1, C9.1, IC1.VDDB, IC2.VO, IC3.HEN, IC3.VCC, IC3.VDD, R4.1
- net +5V: now also C10.2, C11.1, C12.1, C7.2, C8.1, C9.1, CS1.VCC, IC2.VDD1-1, IC2.VDD1-2, X1-2.S; no longer C3.2, C4.1, C5.2, C6.1, IC1.VDD1-1, IC1.VDD1-2, X2-1.S
- net AGND: now also C14.2, C15.2, C16.2, C19.2, C20.2, C25.2, C26.2, C27.2, C29.2, C30.2, C31.2, IC10.V-, IC2.GNDB, IC2.GNDISO, IC3.GND, IC3.GND@1, IC4.DIS, IC4.VSS, IC7.-VS, IC8.-V, IC8.REF, IC9.-VS, R8.1, T1.S, TP1.P$1, X10-2.S, X5-2.S, X6-2.S; no longer C10.2, C11.2, C12.2, C7.2, C8.2, C9.2, IC1.GNDB, IC1.GNDISO, IC2.GND, IC2.GND@1, IC3.DIS, IC3.VSS, R5.2, R6.1, R7.1
- net GND: now also C10.1, C11.2, C12.2, C21.1, C22.2, C3.2, C6.1, C7.1, C8.2, C9.2, CS1.GND, D3.A, IC1.REF, IC2.GND1-1, IC2.GND1-2, IC2.GND1-3, IC2.VIA, IC5.A1, IC5.C, IC6.IN+, R2.1, TP2.P$1, X1-3.S, X3-2.S, X8-2.S; no longer C3.1, C6.2, IC1.GND1-1, IC1.GND1-2, IC1.GND1-3, IC1.VIA, X1-2.S
- net N$10: now also C13.1, C14.1, IC2.VISO, IC3.VI; no longer C7.1, C8.1, IC1.VISO, IC2.VI
- net N$13: now also IC2.VOB, R6.1; no longer IC3.IN-, R3.2
- net N$16: now also C18.2, IC4.AHS, X7-2.S; no longer IC3.LDEL, R7.2
- net N$17: now also C17.2, D1.C, IC4.BHB; no longer C15.2, D2.C, IC3.BHB
- net N$20: now also C18.1, D2.C, IC4.AHB; no longer IC3.OUT, R8.2
- net N$23: now also C17.1, IC4.BHS, X4-2.S; no longer C14.2, D1.C, IC3.AHB
- net N$24: now also IC4.BHO, X4-1.S; no longer IC3.HDEL, R6.2
- net N$28: now also R2.2, R4.1, X2-1.S; no longer R1.2, R2.1, X1-1.S
- net N$29: now also IC4.BLO, X5-1.S; no longer C11.1, IC3.IN+, R4.2, R5.1, R8.1
- net N$30: now also IC2.VIB, R4.2; no longer IC1.VIB, R2.2
- net N$8: now also IC4.DEL, R8.2; no longer IC1.VOB, R3.1
Other:
- note added: "+ -"
- note added: "2.5V"
- note added: "2.5V + 37.5 mV/A"
- note added: "AD8227 operates well even when inputs are near rail voltages want gain ~ 100 to get 1V/A G = 5 + (80k / Rg) Rg = 80k / (G-5) input resistors protect from transients"
- note added: "AGND"
- note added: "AHIGH"
- note added: "ALOW"
- note added: "BHIGH"
- note added: "BLOW"
- note added: "H-bridge control !A->B! / B->A"
- note added: "NOTE: the bypass option/circuit is not shown. Please consult the 'bypass' sheet for guidance"
- note added: "Rsense 10 mOhms"
- note added: "[B]"
- note added: "adjust for 1:1 optocoupling"
- note added: "another option would be to use a LT6105 and put sense resistor on the high side For the inst. amp. I've put Rsense on the low side to allow the FET body diode to protect the input(s) from switching transients."
- note added: "another option would be to use a sense resistor and a LT1999 to generate monitor signal 'directly'"
- note added: "bypass"
- note added: "bypass control 0--10 V 1V = 1A"
- note added: "coil"
- note added: "diode drop"
- note added: "from 10 mOhm sense resistor"
- note added: "galvanically isolated LEM CASR-15 current sensor in series with coil connect all 3 primary turns (Ng = 3) -> 0.24 mOhms"
- note added: "high = VDDB (reg)"
- note added: "high = VISO (unreg)"
- note added: "isolated section floating on lower H-bridge source potential (AGND)"
- note added: "isolated section floating on lower H-bridge source potential (receiver)"
- note added: "nominal <10 mA isolated current quiescent current draw: HIP4082: 4 mA BUF634: 1.5 mA AD8227: 0.5 mA AD820 (x2): 1 mA (2 mA) TOTAL: 8 mA"
- note added: "output molex connectors have 1=gate, 2=source gate protection etc. at FET a good citizen would not twist gate/source wires, input inductance is generally bad!"
- note added: "photocurrent drives IC8 output positive"
- note added: "protection"
- note added: "section referenced to lab potential (GND)"
- note added: "section referenced to lab potential (transmitter)"
- note added: "the bypass circuit is driven "open loop" from the ground-referenced side using a precision matched phototransistor pair. Local feedback on the floating side maintains stability/linearity. Note: you can't bypass more current than is flowing through the H-bridge (duh). Unsure how close you can get before the bypass FET gets too deep into the linear/triode region. [B] If there isn't enough drain-sou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"
- note added: "to bypass FET"
- note added: "want gain ~ 2.67 to get 100mV/A G = 1 + (49.4 k / Rg)"
- note removed: "5V at 125 mA"
- note removed: "control"
- note removed: "high = VDDB (regulated)"
- note removed: "high = VISO (unregulated)"
- note removed: "output molex connectors: A/B different sequence gate protection etc. at FET a good citizen would not twist gate/source wires, input inductance is bad!"
