File: CCM_0019_IXFN_FET_Connector/CCM_0019.brd (EAGLE design)
At the start: 8.1 x 35.6 mm, 7 parts, among them X1 22-23-2021

Commit message: Updated designs for MOT coil control and H-bridge switching
Parts:
- D4: value BZX84B15 -> BZX84B18
Changed lines of the file:
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@@
 <?xml version="1.0" encoding="utf-8"?>
 <!DOCTYPE eagle SYSTEM "eagle.dtd">
-<eagle version="9.0.1">
+<eagle version="9.2.1">
 <drawing>
 <settings>
@@
 <param name="checkStop" value="0"/>
 <param name="checkValues" value="0"/>
+<param name="checkNames" value="1"/>
+<param name="checkWireStubs" value="1"/>
+<param name="checkPolygonWidth" value="0"/>
 <param name="useDiameter" value="13"/>
 <param name="maxErrors" value="50"/>
@@
 </autorouter>
 <elements>
-<element name="D4" library="diode" library_urn="urn:adsk.eagle:library:210" package="SOT23" package3d_urn="urn:adsk.eagle:package:43389@1/2" value="BZX84B15" x="5.842" y="12.446" smashed="yes">
+<element name="D4" library="diode" library_urn="urn:adsk.eagle:library:210" package="SOT23" package3d_urn="urn:adsk.eagle:package:43389@1/2" value="BZX84B18" x="5.842" y="12.446" smashed="yes">
 <attribute name="NAME" x="6.731" y="13.589" size="0.6096" layer="25" font="vector" ratio="15"/>
 <attribute name="VALUE" x="3.937" y="9.271" size="1.27" layer="27"/>
@@
 <attribute name="VALUE" x="1.27" y="9.779" size="1.27" layer="27"/>
 </element>
-<element name="H1" library="noah" package="4.2-PAD-SMALL" value="4.2-PAD-SMALL" x="4.318" y="5.08"/>
-<element name="H2" library="noah" package="4.2-PAD-SMALL" value="4.2-PAD-SMALL" x="4.318" y="20.066"/>
+<element name="H1" library="noah" package="4.2-PAD-SMALL" value="4.2-PAD-SMALL" x="4.318" y="5.08" smashed="yes"/>
+<element name="H2" library="noah" package="4.2-PAD-SMALL" value="4.2-PAD-SMALL" x="4.318" y="20.066" smashed="yes"/>
 </elements>
 <signals>
@@
 </signal>
 </signals>
+<mfgpreviewcolors>
+<mfgpreviewcolor name="soldermaskcolor" color="0xC8008000"/>
+<mfgpreviewcolor name="silkscreencolor" color="0xFFFEFEFE"/>
+<mfgpreviewcolor name="backgroundcolor" color="0xFF282828"/>
+<mfgpreviewcolor name="coppercolor" color="0xFFFFBF00"/>
+<mfgpreviewcolor name="substratecolor" color="0xFF786E46"/>
+</mfgpreviewcolors>
 </board>
 </drawing>
