File: CCM_0008_Precision_FET_Driver/revB/CCM_0008.brd (EAGLE design)
At the start: 41.9 x 69.8 mm, 58 parts, among them IC1 AD8226, IC2 AD825, IC3 AD8226, IC4 AD825, X1 22-23-2021, X2 22-23-2021, X3 22-23-2041, X5 22-23-2021

Commit message: Updated component values on circuits used for MOT coil driving and H-bridges.
Parts:
- C20: value 1n -> 10n
- C24: value 20p -> 100p
- R8: value 200k -> 100k
Changed lines of the file:
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@@
 <attribute name="VALUE" x="18.923" y="48.514" size="0.6096" layer="27" font="vector" ratio="20" rot="R90"/>
 </element>
-<element name="C24" library="acrooptics" package="0603" value="20p" x="17.145" y="53.6575" smashed="yes" rot="R270">
+<element name="C24" library="acrooptics" package="0603" value="100p" x="17.145" y="53.6575" smashed="yes" rot="R270">
 <attribute name="NAME" x="16.383" y="55.372" size="0.6096" layer="25" font="vector" ratio="15"/>
 <attribute name="VALUE" x="15.367" y="55.3085" size="0.6096" layer="27" font="vector" ratio="20" rot="R270"/>
 </element>
-<element name="C20" library="acrooptics" package="0603" value="1n" x="15.24" y="50.165" smashed="yes" rot="R270">
+<element name="C20" library="acrooptics" package="0603" value="10n" x="15.24" y="50.165" smashed="yes" rot="R270">
 <attribute name="NAME" x="14.605" y="52.07" size="0.6096" layer="25" font="vector" ratio="15"/>
 <attribute name="VALUE" x="13.462" y="51.816" size="0.6096" layer="27" font="vector" ratio="20" rot="R270"/>
 </element>
-<element name="R8" library="rcl" library_urn="urn:adsk.eagle:library:334" package="RTRIM3296W" package3d_urn="urn:adsk.eagle:package:23739/1" value="200k" x="10.795" y="42.545" smashed="yes" rot="R90">
+<element name="R8" library="rcl" library_urn="urn:adsk.eagle:library:334" package="RTRIM3296W" package3d_urn="urn:adsk.eagle:package:23739/1" value="100k" x="10.795" y="42.545" smashed="yes" rot="R90">
 <attribute name="NAME" x="15.7565" y="42.2105" size="0.6096" layer="25" font="vector" ratio="15"/>
 <attribute name="SPICEMODEL" value="X" x="10.795" y="42.545" size="1.778" layer="27" rot="R90" display="off"/>
