File: CCM_0010_Floating_H_Bridge/revC/CCM_0010.brd (EAGLE design)
At the start: 50.8 x 76.2 mm, 65 parts, among them IC1 ADUM5230, IC10 LT1097, IC2 UAL78L12, IC3 HIP4082, IC8 HCNR200-300E, IC9 LT1097, T1 2N7002, T2 MMBT3906, X1 22-23-2041, X2 22-23-2021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

Commit message: Updated component values on circuits used for MOT coil driving and H-bridges.
Parts:
- IC10: value LT1097 -> AD820
Changed lines of the file:
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@@
 <attribute name="VALUE" x="34.544" y="62.484" size="0.6096" layer="27" font="vector" ratio="20" rot="R270"/>
 </element>
-<element name="IC10" library="linear" library_urn="urn:adsk.eagle:library:262" package="SO08" package3d_urn="urn:adsk.eagle:package:16404/2" value="LT1097" x="41.275" y="50.165" smashed="yes">
+<element name="IC10" library="linear" library_urn="urn:adsk.eagle:library:262" package="SO08" package3d_urn="urn:adsk.eagle:package:16404/2" value="AD820" x="41.275" y="50.165" smashed="yes">
 <attribute name="NAME" x="43.8785" y="52.5145" size="0.6096" layer="25" font="vector" ratio="15"/>
 <attribute name="VALUE" x="45.212" y="48.26" size="1.27" layer="27" rot="R90"/>
