File: CCM_0010_Floating_H_Bridge/revC/CCM_0010.sch (EAGLE design)
At the start: 65 parts, among them IC1 ADUM5230, IC10 LT1097, IC2 UAL78L12, IC3 HIP4082, IC8 HCNR200-300E, IC9 LT1097, T1 2N7002, T2 MMBT3906, X1 22-23-2041, X2 22-23-2021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

Commit message: Updated component values on circuits used for MOT coil driving and H-bridges.
Parts:
- IC10: value LT1097 -> AD820
Changed lines of the file:
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@@
 <setting verticaltext="up"/>
 </settings>
-<grid distance="0.025" unitdist="inch" unit="inch" style="lines" multiple="4" display="yes" altdistance="0.01" altunitdist="inch" altunit="inch"/>
+<grid distance="0.1" unitdist="inch" unit="inch" style="lines" multiple="1" display="no" altdistance="0.01" altunitdist="inch" altunit="inch"/>
 <layers>
 <layer number="1" name="Top" color="4" fill="1" visible="no" active="no"/>
@@
 <part name="C33" library="acrooptics" deviceset="C" device="0603" value="DNI"/>
 <part name="AGND12" library="supply1" library_urn="urn:adsk.eagle:library:371" deviceset="AGND" device=""/>
-<part name="IC10" library="linear" library_urn="urn:adsk.eagle:library:262" deviceset="OP07*" device="R" package3d_urn="urn:adsk.eagle:package:16404/2" technology="C" value="LT1097"/>
+<part name="IC10" library="linear" library_urn="urn:adsk.eagle:library:262" deviceset="OP07*" device="R" package3d_urn="urn:adsk.eagle:package:16404/2" technology="C" value="AD820"/>
 <part name="C32" library="acrooptics" deviceset="C" device="0603" value="DNI"/>
 <part name="IC9" library="linear" library_urn="urn:adsk.eagle:library:262" deviceset="OP07*" device="R" package3d_urn="urn:adsk.eagle:package:16404/2" technology="C" value="LT1097"/>

Commit message: many changes
Other:
- note added: "charge pump diodes (D1/D2) should be Schottky (fast), rated for > 60V bootstrap capacitors (C15/C16) should be > 10x FET gate-source capacitance IXFN180N15P FET has Cgs = 7nF IXFN360N10P FET has Cgs = 36nF"
- note added: "nominal <10 mA isolated current expected quiescent current draw: HIP4082: 4 mA AD820 (next sheet): 1 mA"
- note added: "output molex connectors have 1=gate, 2=source"
- note removed: "charge pump diodes (D1/D2) should be Schottky (fast), rated for > 60V bootstrap capacitors (C14/C15) should be > 10x FET gate-source capacitance IXFN180N15P FET has Cgs = 7nF"
- note removed: "nominal <10 mA isolated current expected quiescent current draw: HIP4082: 4 mA LT1097: 1 mA"
- note removed: "output molex connectors have 1=gate, 2=source gate protection etc. at FET a good citizen would not twist gate/source wires, input inductance is generally bad!"
Changed lines of the file:
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@@
 <?xml version="1.0" encoding="utf-8"?>
 <!DOCTYPE eagle SYSTEM "eagle.dtd">
-<eagle version="9.3.1">
+<eagle version="9.5.1">
 <drawing>
 <settings>
@@
 <setting verticaltext="up"/>
 </settings>
-<grid distance="0.1" unitdist="inch" unit="inch" style="lines" multiple="1" display="no" altdistance="0.01" altunitdist="inch" altunit="inch"/>
+<grid distance="0.025" unitdist="inch" unit="inch" style="lines" multiple="4" display="yes" altdistance="0.01" altunitdist="inch" altunit="inch"/>
 <layers>
 <layer number="1" name="Top" color="4" fill="1" visible="no" active="no"/>
@@
 <text x="132.715" y="113.665" size="1.778" layer="97">high = VISO (unreg)</text>
 <text x="132.715" y="109.855" size="1.778" layer="97">high = VDDB (reg)</text>
-<text x="218.44" y="63.5" size="1.778" layer="97">output molex connectors
-have 1=gate, 2=source
-gate protection etc. at FET
-a good citizen would not twist
-gate/source wires, input
-inductance is generally bad!</text>
+<text x="220.98" y="73.66" size="1.778" layer="97">output molex connectors
+have 1=gate, 2=source</text>
 <text x="170.18" y="63.5" size="1.778" layer="97">charge pump diodes (D1/D2) should
 be Schottky (fast), rated for &gt; 60V
-bootstrap capacitors (C14/C15) should
+bootstrap capacitors (C15/C16) should
 be  &gt; 10x FET gate-source capacitance
-IXFN180N15P FET has Cgs = 7nF</text>
+IXFN180N15P FET has Cgs = 7nF
+IXFN360N10P FET has Cgs = 36nF</text>
 <text x="116.84" y="63.5" size="1.778" layer="97">nominal &lt;10 mA isolated current
 expected quiescent current draw:
 HIP4082: 4 mA
-LT1097: 1 mA</text>
+AD820 (next sheet): 1 mA</text>
 <text x="239.395" y="125.095" size="1.778" layer="97">BHIGH</text>
 <text x="239.395" y="120.015" size="1.778" layer="97">BLOW</text>
