File: CCM_0020_Floating_Leakage_Monitor/CCM_0020_receiver.sch (EAGLE design)
At the start: 91 parts, among them IC1 AD8656R, IC10 LF356D, IC11 LF356D, IC2 LM311D, IC3 LT1495, IC4 741G00, IC5 741G04, IC6 741G04, IC7 741G04, IC8 AD820R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

Commit message: Simplified leakage monitor receiver.
Parts:
- removed R7: 30k, acrooptics:R0603
- removed R9: 20k, acrooptics:R0603
- D1: value LM4040-2.5V -> MAX6006
Connections:
- removed net N$9: IC2.-IN, R7.2, R9.1
- net GND: no longer R9.2
- net N$14: now also IC2.-IN; no longer R7.1
Other:
- note added: "1.25V"
- note removed: "1V"
